Commit message: change controller arg order and update models

File: src/Models/urdf/planar_atlas_with_walls.urdf (robot description, URDF)
Before this commit: robot atlas, 66 links, 65 joints
Links:
- removed link floating_base_dummy
Joints:
- removed joint floating_base_dummy_to_pelvis
- joint floating_base: axis 0 -1 0 -> 1 0 0; child floating_base_dummy -> pelvis; origin rpy=0 0 1.5707963267948966 -> rpy=0 0 0
- joint l_arm_mwx: type revolute -> fixed
- joint l_arm_uwy: type revolute -> fixed
- joint r_arm_mwx: type revolute -> fixed
- joint r_arm_uwy: type revolute -> fixed
