Commit message: rotate box atlas to better match true atlas state

File: src/Models/urdf/box_atlas.urdf (robot description, URDF)
Before this commit: robot BoxAtlas, 12 links, 11 joints
Joints:
- removed joint root_to_wall
- added joint floor_to_wall: type fixed, parent floor, child wall
- joint floating_base: parent root -> floor
- joint root_to_floor: origin (none) -> rpy=0 0 -1.5707963267948966

Commit message: update box_atlas.urdf to more closely match the real robot

File: src/Models/urdf/box_atlas.urdf (robot description, URDF)
Before this commit: robot BoxAtlas, 12 links, 11 joints
Links:
- removed link core
- removed link lf
- removed link lf_dummy
- removed link lh
- removed link lh_dummy
- removed link rf
- removed link rf_dummy
- removed link rh
- removed link rh_dummy
- added link floating_base_dummy, mass 0.0
- added link l_foot_sole, mass 0.2; collision sphere radius=0; visual cylinder length=0.475 radius=0.02
- added link l_foot_sole_dummy, mass 0.0; visual cylinder length=0.475 radius=0.03; visual sphere radius=0.05
- added link l_hand_mount, mass 0.05; collision sphere radius=0; visual cylinder length=0.4 radius=0.02
- added link l_hand_mount_dummy, mass 0.0; visual cylinder length=0.4 radius=0.03; visual sphere radius=0.05
- added link pelvis, mass 1.0; visual box size=0.05 0.4 0.55
- added link r_foot_sole, mass 0.2; collision sphere radius=0; visual cylinder length=0.475 radius=0.02
- added link r_foot_sole_dummy, mass 0.0; visual cylinder length=0.475 radius=0.03; visual sphere radius=0.05
- added link r_hand_mount, mass 0.05; collision sphere radius=0; visual cylinder length=0.4 radius=0.02
- added link r_hand_mount_dummy, mass 0.0; visual cylinder length=0.4 radius=0.03; visual sphere radius=0.05
- link floor: geometry collision box size=1 3 0.1; collision plane normal=0 0 1
- link wall: geometry collision box size=1 0.1 2.2; collision plane normal=0 -1 0
Joints:
- removed joint core_to_lf_extension
- removed joint core_to_lf_rotation
- removed joint core_to_lh_extension
- removed joint core_to_lh_rotation
- removed joint core_to_rf_extension
- removed joint core_to_rf_rotation
- removed joint core_to_rh_extension
- removed joint core_to_rh_rotation
- added joint floating_base_dummy_to_pelvis: type fixed, parent floating_base_dummy, child pelvis, origin rpy=0 0 -1.5707963267948966
- added joint pelvis_to_l_foot_sole_extension: type prismatic, parent l_foot_sole_dummy, child l_foot_sole, origin xyz=0 0 0, axis 0 0 1, limit lower=0.45 upper=0.9 effort=20 velocity=100
- added joint pelvis_to_l_foot_sole_rotation: type revolute, parent pelvis, child l_foot_sole_dummy, origin xyz=0 0.11 0 rpy=3.1415926535897 0 0, axis 1 0 0, limit lower=-0.05 upper=0.785398 effort=10 velocity=100
- added joint pelvis_to_l_hand_mount_extension: type prismatic, parent l_hand_mount_dummy, child l_hand_mount, origin xyz=0 0 0, axis 0 0 1, limit lower=0.375 upper=0.75 effort=2 velocity=100
- added joint pelvis_to_l_hand_mount_rotation: type revolute, parent pelvis, child l_hand_mount_dummy, origin xyz=0 0.3 0.45 rpy=3.1415926535897 0 0, axis 1 0 0, limit lower=0 upper=1.6708 effort=2 velocity=100
- added joint pelvis_to_r_foot_sole_extension: type prismatic, parent r_foot_sole_dummy, child r_foot_sole, origin xyz=0 0 0, axis 0 0 1, limit lower=0.45 upper=0.9 effort=20 velocity=100
- added joint pelvis_to_r_foot_sole_rotation: type revolute, parent pelvis, child r_foot_sole_dummy, origin xyz=0 -0.11 0 rpy=3.1415926535897 0 0, axis -1 0 0, limit lower=-0.05 upper=0.785398 effort=10 velocity=100
- added joint pelvis_to_r_hand_mount_extension: type prismatic, parent r_hand_mount_dummy, child r_hand_mount, origin xyz=0 0 0, axis 0 0 1, limit lower=0.375 upper=0.75 effort=2 velocity=100
- added joint pelvis_to_r_hand_mount_rotation: type revolute, parent pelvis, child r_hand_mount_dummy, origin xyz=0 -0.3 0.45 rpy=-3.1415926535897 0 0, axis -1 0 0, limit lower=0 upper=1.6708 effort=2 velocity=100
- joint floating_base: child core -> floating_base_dummy; origin (none) -> rpy=0 0 1.5707963267948966; parent floor -> root
- joint root_to_floor: origin rpy=0 0 -1.5707963267948966 -> (none)

Commit message: update joint limits

File: src/Models/urdf/box_atlas.urdf (robot description, URDF)
Before this commit: robot BoxAtlas, 13 links, 12 joints
Joints:
- joint pelvis_to_l_foot_sole_extension: limit lower=0.45 upper=0.9 effort=20 velocity=100 -> lower=0.475 upper=0.95 effort=20 velocity=100
- joint pelvis_to_l_hand_mount_extension: limit lower=0.375 upper=0.75 effort=2 velocity=100 -> lower=0.4 upper=0.8 effort=2 velocity=100
- joint pelvis_to_r_foot_sole_extension: limit lower=0.45 upper=0.9 effort=20 velocity=100 -> lower=0.475 upper=0.95 effort=20 velocity=100
- joint pelvis_to_r_hand_mount_extension: limit lower=0.375 upper=0.75 effort=2 velocity=100 -> lower=0.4 upper=0.8 effort=2 velocity=100

Commit message: fix floor position

File: src/Models/urdf/box_atlas.urdf (robot description, URDF)
Before this commit: robot BoxAtlas, 13 links, 12 joints
Links:
- link floor: geometry collision box size=1 3 0.1; collision plane normal=0 0 1

Commit message: more realistic box atlas inertias

File: src/Models/urdf/box_atlas.urdf (robot description, URDF)
Before this commit: robot BoxAtlas, 13 links, 12 joints
Links:
- link l_foot_sole: mass 0.2 -> 7.05
- link l_foot_sole_dummy: mass 0.0 -> 9.1
- link l_hand_mount: mass 0.05 -> 7.06
- link l_hand_mount_dummy: mass 0.0 -> 8.285
- link pelvis: mass 1.0 -> 112.12
- link r_foot_sole: mass 0.2 -> 7.05
- link r_foot_sole_dummy: mass 0.0 -> 9.1
- link r_hand_mount: mass 0.05 -> 7.06
- link r_hand_mount_dummy: mass 0.0 -> 8.285
Joints:
- joint pelvis_to_l_foot_sole_extension: axis 0 0 1 -> 0 0 -1; limit lower=0.475 upper=0.95 effort=20 velocity=100 -> lower=0.475 upper=0.95 effort=3000 velocity=100; origin xyz=0 0 0 -> xyz=0 0 0 rpy=3.1415926535897 0 0
- joint pelvis_to_l_foot_sole_rotation: limit lower=-0.05 upper=0.785398 effort=10 velocity=100 -> lower=-0.05 upper=0.785398 effort=530 velocity=100
- joint pelvis_to_l_hand_mount_extension: axis 0 0 1 -> 0 1 0; limit lower=0.4 upper=0.8 effort=2 velocity=100 -> lower=0.4 upper=0.8 effort=500 velocity=100; origin xyz=0 0 0 -> xyz=0 0 0 rpy=1.5707963267948966 0 -1.5707963267948966
- joint pelvis_to_l_hand_mount_rotation: limit lower=0 upper=1.6708 effort=2 velocity=100 -> lower=0 upper=1.6708 effort=100 velocity=100
- joint pelvis_to_r_foot_sole_extension: axis 0 0 1 -> 0 0 -1; limit lower=0.475 upper=0.95 effort=20 velocity=100 -> lower=0.475 upper=0.95 effort=3000 velocity=100; origin xyz=0 0 0 -> xyz=0 0 0 rpy=3.1415926535897 0 0
- joint pelvis_to_r_foot_sole_rotation: limit lower=-0.05 upper=0.785398 effort=10 velocity=100 -> lower=-0.05 upper=0.785398 effort=530 velocity=100
- joint pelvis_to_r_hand_mount_extension: axis 0 0 1 -> 0 1 0; limit lower=0.4 upper=0.8 effort=2 velocity=100 -> lower=0.4 upper=0.8 effort=500 velocity=100; origin xyz=0 0 0 -> xyz=0 0 0 rpy=1.5707963267948966 0 1.5707963267948966
- joint pelvis_to_r_hand_mount_rotation: limit lower=0 upper=1.6708 effort=2 velocity=100 -> lower=0 upper=1.6708 effort=100 velocity=100

Commit message: better box atlas defaults

File: src/Models/urdf/box_atlas.urdf (robot description, URDF)
Before this commit: robot BoxAtlas, 13 links, 12 joints
Joints:
- joint pelvis_to_l_foot_sole_extension: limit lower=0.475 upper=0.95 effort=3000 velocity=100 -> lower=0.475 upper=0.95 effort=2100 velocity=100
- joint pelvis_to_r_foot_sole_extension: limit lower=0.475 upper=0.95 effort=3000 velocity=100 -> lower=0.475 upper=0.95 effort=2100 velocity=100

Commit message: penalize vdot, not u

File: src/Models/urdf/box_atlas.urdf (robot description, URDF)
Before this commit: robot BoxAtlas, 13 links, 12 joints
Joints:
- joint floating_base: limit (none) -> effort=0

File: src/Models/urdf/planar_atlas_with_walls.urdf (robot description, URDF)
Before this commit: robot atlas, 66 links, 65 joints
Joints:
- joint back_bkx: type revolute -> fixed
- joint back_bky: type revolute -> fixed
- joint back_bkz: type revolute -> fixed
- joint floating_base: limit (none) -> effort=0
- joint l_leg_hpz: type revolute -> fixed
- joint neck_ay: type revolute -> fixed
- joint r_leg_hpz: type revolute -> fixed

Commit message: restore older box atlas masses

File: src/Models/urdf/box_atlas.urdf (robot description, URDF)
Before this commit: robot BoxAtlas, 13 links, 12 joints
Links:
- link l_foot_sole: mass 7.05 -> 0.2
- link l_foot_sole_dummy: mass 9.1 -> 0.0
- link l_hand_mount: mass 7.06 -> 0.05
- link l_hand_mount_dummy: mass 8.285 -> 0.0
- link pelvis: mass 112.12 -> 1.0
- link r_foot_sole: mass 7.05 -> 0.2
- link r_foot_sole_dummy: mass 9.1 -> 0.0
- link r_hand_mount: mass 7.06 -> 0.05
- link r_hand_mount_dummy: mass 8.285 -> 0.0
Joints:
- joint pelvis_to_l_foot_sole_extension: limit lower=0.475 upper=0.95 effort=2100 velocity=100 -> lower=0.475 upper=0.95 effort=20 velocity=100
- joint pelvis_to_l_foot_sole_rotation: limit lower=-0.05 upper=0.785398 effort=530 velocity=100 -> lower=-0.05 upper=0.785398 effort=10 velocity=100
- joint pelvis_to_l_hand_mount_extension: axis 0 1 0 -> 0 0 1; limit lower=0.4 upper=0.8 effort=500 velocity=100 -> lower=0.4 upper=0.8 effort=2 velocity=100; origin xyz=0 0 0 rpy=1.5707963267948966 0 -1.5707963267948966 -> xyz=0 0 0
- joint pelvis_to_l_hand_mount_rotation: limit lower=0 upper=1.6708 effort=100 velocity=100 -> lower=0 upper=1.6708 effort=2 velocity=100
- joint pelvis_to_r_foot_sole_extension: limit lower=0.475 upper=0.95 effort=2100 velocity=100 -> lower=0.475 upper=0.95 effort=20 velocity=100
- joint pelvis_to_r_foot_sole_rotation: limit lower=-0.05 upper=0.785398 effort=530 velocity=100 -> lower=-0.05 upper=0.785398 effort=10 velocity=100
- joint pelvis_to_r_hand_mount_extension: axis 0 1 0 -> 0 0 1; limit lower=0.4 upper=0.8 effort=500 velocity=100 -> lower=0.4 upper=0.8 effort=2 velocity=100; origin xyz=0 0 0 rpy=1.5707963267948966 0 1.5707963267948966 -> xyz=0 0 0
- joint pelvis_to_r_hand_mount_rotation: limit lower=0 upper=1.6708 effort=100 velocity=100 -> lower=0 upper=1.6708 effort=2 velocity=100
